Commit message: gazebo.launch.py working fine. friction coefficients are haolding the arm

File: src/jetrover_description/urdf/arm.urdf.xacro (robot description, xacro)
@@ -140,4 +140,7 @@
       effort="1000"
       velocity="10" />
+    <dynamics
+      damping="0.5"
+      friction="0.1"/>
   </joint>
   <link
@@ -194,4 +197,7 @@
       effort="1000"
       velocity="10" />
+    <dynamics
+      damping="0.5"
+      friction="0.1"/>
   </joint>
   <link
@@ -248,4 +254,7 @@
       effort="1000"
       velocity="10" />
+    <dynamics
+      damping="0.5"
+      friction="0.1"/>
   </joint>
   <link
@@ -351,4 +360,7 @@
       effort="1000"
       velocity="10" />
+    <dynamics
+      damping="0.5"
+      friction="0.1"/>
   </joint>
   <link

File: src/jetrover_description/urdf/hiwonder_jetrover.xacro (robot description, xacro)
@@ -1,4 +1,6 @@
 <?xml version="1.0" encoding="utf-8"?>
 <robot name="hiwonder" xmlns:xacro="http://ros.org/wiki/xacro">
+    <!-- change default to True to enable ROS2 control : Using it false to check if gazebo is working correctly -->
+    <xacro:arg name="enable_ros2_control" default="false"/>
     <xacro:property name="lidar"        value="$(env LIDAR_TYPE)"/>
     <xacro:property name="machine"      value="$(env MACHINE_TYPE)"/>
@@ -32,5 +34,7 @@
     <!--<xacro:include filename="$(find jetrover_description)/urdf/gripper.transmission.xacro"/> ROS1 framework-->
     <!-- ROS 2 control interfaces -->
-    <xacro:include filename="$(find jetrover_description)/urdf/hiwonder_jetrover_ros2control.xacro"/>
+    <xacro:if value="$(arg enable_ros2_control)">
+        <xacro:include filename="$(find jetrover_description)/urdf/hiwonder_jetrover_ros2control.xacro"/>
+    </xacro:if>
     <!-- Gazebo physics and plugins -->
     <xacro:include filename="$(find jetrover_description)/urdf/hiwonder_jetrover_gazebo.xacro"/>

File: src/jetrover_description/urdf/hiwonder_jetrover_gazebo.xacro (robot description, xacro)
@@ -1,43 +1,83 @@
 <?xml version="1.0"?>
 <robot name="hiwonder" xmlns:xacro="http://www.ros.org/wiki/xacro">
-  <!-- Friction for the four Mecanum wheels -->
-  <gazebo reference="wheel_left_front_link">
-    <mu1>1.0</mu1>
-    <mu2>1.0</mu2>
-    <kp>1000000.0</kp>
-    <kd>100.0</kd>
-    <minDepth>0.001</minDepth>
-    <maxVel>0.1</maxVel>
-  </gazebo>
-  <gazebo reference="wheel_left_back_link">
-    <mu1>1.0</mu1>
-    <mu2>1.0</mu2>
-    <kp>1000000.0</kp>
-    <kd>100.0</kd>
-    <minDepth>0.001</minDepth>
-    <maxVel>0.1</maxVel>
-  </gazebo>
-  <gazebo reference="wheel_right_front_link">
-    <mu1>1.0</mu1>
-    <mu2>1.0</mu2>
-    <kp>1000000.0</kp>
-    <kd>100.0</kd>
-    <minDepth>0.001</minDepth>
-    <maxVel>0.1</maxVel>
-  </gazebo>
-  <gazebo reference="wheel_right_back_link">
-    <mu1>1.0</mu1>
-    <mu2>1.0</mu2>
-    <kp>1000000.0</kp>
-    <kd>100.0</kd>
-    <minDepth>0.001</minDepth>
-    <maxVel>0.1</maxVel>
-  </gazebo>
-  <!-- ROS 2 Control plugin for Gazebo Harmonic -->
-  <gazebo>
-    <plugin
-      filename="libgz_ros2_control-system.so" name="gz_ros2_control::GazeboSimROS2ControlPlugin">
-      <parameters> $(find jetrover_description)/config/controllers.yaml </parameters>
-    </plugin>
-  </gazebo>
+  <!-- Reusable Gazebo contact-friction settings -->
+  <xacro:macro name="contact_friction" params="link_name mu_value">
+    <gazebo reference="${link_name}">
+      <mu1>${mu_value}</mu1>
+      <mu2>${mu_value}</mu2>
+      <kp>1000000.0</kp>
+      <kd>100.0</kd>
+      <minDepth>0.001</minDepth>
+      <maxVel>0.1</maxVel>
+    </gazebo>
+  </xacro:macro>
+  <!-- Mecanum wheels -->
+  <xacro:contact_friction
+      link_name="wheel_left_front_link"
+      mu_value="1.0"/>
+  <xacro:contact_friction
+      link_name="wheel_left_back_link"
+      mu_value="1.0"/>
+  <xacro:contact_friction
+      link_name="wheel_right_front_link"
+      mu_value="1.0"/>
+  <xacro:contact_friction
+      link_name="wheel_right_back_link"
+      mu_value="1.0"/>
+  <!-- Arm links -->
+  <xacro:contact_friction
+    link_name="link1"
+    mu_value="1.0"/>
+  <xacro:contact_friction
+    link_name="servo_link1"
+    mu_value="1.0"/>
+  <xacro:contact_friction
+    link_name="link2"
+    mu_value="1.0"/>
+  <xacro:contact_friction
+    link_name="link3"
+    mu_value="1.0"/>
+  <xacro:contact_friction
+    link_name="link4"
+    mu_value="1.0"/>
+  <xacro:contact_friction
+    link_name="servo_link2"
+    mu_value="1.0"/>
+  <xacro:contact_friction
+    link_name="link5"
+    mu_value="1.0"/>
+  <xacro:contact_friction
+    link_name="gripper_link"
+    mu_value="1.0"/>
+  <!-- Gripper links -->
+  <xacro:contact_friction
+    link_name="r_link"
+    mu_value="1.0"/>
+  <xacro:contact_friction
+    link_name="r_in_link"
+    mu_value="1.0"/>
+  <xacro:contact_friction
+    link_name="r_out_link"
+    mu_value="1.0"/>
+  <xacro:contact_friction
+    link_name="l_link"
+    mu_value="1.0"/>
+  <xacro:contact_friction
+    link_name="l_in_link"
+    mu_value="1.0"/>
+  <xacro:contact_friction
+    link_name="l_out_link"
+    mu_value="1.0"/>
+  <!-- Enable ROS 2 Control later -->
+  <xacro:if value="$(arg enable_ros2_control)">
+    <gazebo>
+      <plugin
+        filename="libgz_ros2_control-system.so"
+        name="gz_ros2_control::GazeboSimROS2ControlPlugin">
+        <parameters>
+          $(find jetrover_description)/config/controllers.yaml
+        </parameters>
+      </plugin>
+    </gazebo>
+  </xacro:if>
 </robot>
